Commit message: update shapenet block ploygons v2

File: multiworld/envs/pybullet/assets/blocks/train/blk11/obj.urdf (robot description, URDF)
Before this commit: robot block, 1 links, 0 joints
Links:
- link block_base_link: geometry collision mesh filename=12.STL scale=1 1 1; visual mesh filename=12.STL scale=1 1 1

File: multiworld/envs/pybullet/assets/blocks/train/blk12/obj.urdf (robot description, URDF)
Before this commit: robot block, 1 links, 0 joints
Links:
- link block_base_link: geometry collision mesh filename=13.STL scale=1 1 1; visual mesh filename=13.STL scale=1 1 1

File: multiworld/envs/pybullet/assets/blocks/train/blk13/obj.urdf (robot description, URDF)
Before this commit: robot block, 1 links, 0 joints
Links:
- link block_base_link: geometry collision mesh filename=14.STL scale=1 1 1; visual mesh filename=14.STL scale=1 1 1

File: multiworld/envs/pybullet/assets/ploygons/train/blk19/obj.urdf (robot description, URDF)
Before this commit: robot block, 1 links, 0 joints
Links:
- link block_base_link: geometry collision mesh filename=21.STL scale=1 1 1; visual mesh filename=21.STL scale=1 1 1

File: multiworld/envs/pybullet/assets/ploygons/train/blk20/obj.urdf (robot description, URDF)
Before this commit: robot block, 1 links, 0 joints
Links:
- link block_base_link: geometry collision mesh filename=22.STL scale=1 1 1; visual mesh filename=22.STL scale=1 1 1

File: multiworld/envs/pybullet/assets/ploygons/train/blk21/obj.urdf (robot description, URDF)
Before this commit: robot block, 1 links, 0 joints
Links:
- link block_base_link: geometry collision mesh filename=23.STL scale=1 1 1; visual mesh filename=23.STL scale=1 1 1

File: multiworld/envs/pybullet/assets/ploygons/train/blk22/obj.urdf (robot description, URDF)
Before this commit: robot block, 1 links, 0 joints
Links:
- link block_base_link: geometry collision mesh filename=24.STL scale=1 1 1; visual mesh filename=24.STL scale=1 1 1

File: multiworld/envs/pybullet/assets/ploygons/train/blk23/obj.urdf (robot description, URDF)
Before this commit: robot block, 1 links, 0 joints
Links:
- link block_base_link: geometry collision mesh filename=25.STL scale=1 1 1; visual mesh filename=25.STL scale=1 1 1

File: multiworld/envs/pybullet/assets/ploygons/train/blk24/obj.urdf (robot description, URDF)
Before this commit: robot block, 1 links, 0 joints
Links:
- link block_base_link: geometry collision mesh filename=26.STL scale=1 1 1; visual mesh filename=26.STL scale=1 1 1

File: multiworld/envs/pybullet/assets/ploygons/train/blk25/obj.urdf (robot description, URDF)
Before this commit: robot block, 1 links, 0 joints
Links:
- link block_base_link: geometry collision mesh filename=27.STL scale=1 1 1; visual mesh filename=27.STL scale=1 1 1
